File: shupito23/shupito.brd (EAGLE design)
At the start: 41.9 x 23.5 mm, 92 parts, among them IC2 74LVC1T45, IC3 74LVC1T45, IC4 74LVC1T45, IC5 74LVC1T45, IC6 ATXMEGA32A4U-AU, IC7 TPS73033DBV, Q1 BC807W-1907646, Q10 PMF280UN,115-1758094, Q11 PDTC123YU-1757992, Q2 NX2301P-1894738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

Commit message: shupito23: Selected better transistors for the rst pin.
Parts:
- Q6, Q9: value DTA144-1680214 -> PDTA114TU-8736731
Changed lines of the file:
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@@
 <grid distance="0.025" unitdist="inch" unit="mm" style="lines" multiple="1" display="yes" altdistance="3.125" altunitdist="mil" altunit="inch"/>
 <layers>
-<layer number="1" name="Top" color="4" fill="1" visible="yes" active="yes"/>
+<layer number="1" name="Top" color="4" fill="1" visible="no" active="yes"/>
 <layer number="16" name="Bottom" color="1" fill="1" visible="yes" active="yes"/>
 <layer number="17" name="Pads" color="2" fill="1" visible="yes" active="yes"/>
@@
 <layer number="21" name="tPlace" color="7" fill="1" visible="no" active="yes"/>
 <layer number="22" name="bPlace" color="7" fill="1" visible="no" active="yes"/>
-<layer number="23" name="tOrigins" color="15" fill="1" visible="yes" active="yes"/>
+<layer number="23" name="tOrigins" color="15" fill="1" visible="no" active="yes"/>
 <layer number="24" name="bOrigins" color="15" fill="1" visible="yes" active="yes"/>
-<layer number="25" name="tNames" color="7" fill="1" visible="yes" active="yes"/>
-<layer number="26" name="bNames" color="7" fill="1" visible="yes" active="yes"/>
+<layer number="25" name="tNames" color="7" fill="1" visible="no" active="yes"/>
+<layer number="26" name="bNames" color="7" fill="1" visible="no" active="yes"/>
 <layer number="27" name="tValues" color="7" fill="1" visible="no" active="yes"/>
 <layer number="28" name="bValues" color="7" fill="1" visible="no" active="yes"/>
@@
 <element name="R1" library="rcl" package="R0603" value="330" x="5.08" y="19.05" rot="MR270"/>
 <element name="R2" library="rcl" package="R0603" value="6k8" x="18.415" y="6.35" rot="MR0"/>
-<element name="Q9" library="transistors" package="SOT323" value="DTA144-1680214" x="18.415" y="17.78" rot="MR0"/>
+<element name="Q9" library="transistors" package="SOT323" value="PDTA114TU-8736731" x="18.415" y="17.78" rot="MR0"/>
 <element name="R13" library="rcl" package="R0603" value="22k 1%" x="26.9875" y="8.89" rot="MR0"/>
 <element name="R14" library="rcl" package="R0603" value="1k5 1%" x="26.035" y="11.43" rot="MR270"/>
 <element name="IC6" library="xmega" package="TQFP44" value="ATXMEGA32A4U-AU" x="23.495" y="10.795" rot="R270"/>
 <element name="X2" library="usb" package="USB-MICRO-B-BOTTOM-MOLEX" value="USB-MICRO-B-BOTTOM" x="40.48125" y="12.065" rot="R180"/>
-<element name="Q6" library="transistors" package="SOT323" value="DTA144-1680214" x="7.62" y="19.685" rot="MR270"/>
+<element name="Q6" library="transistors" package="SOT323" value="PDTA114TU-8736731" x="7.62" y="19.685" rot="MR270"/>
 <element name="Q11" library="transistors" package="SOT323" value="PDTC123YU-1757992" x="10.795" y="17.78" rot="MR0"/>
 <element name="C2" library="rcl" package="C0603K" value="10n" x="27.94" y="11.43" rot="MR270"/>
