File: shupito23/shupito.brd (EAGLE design)
At the start: 41.9 x 23.5 mm, 92 parts, among them IC2 74LVC1T45, IC3 74LVC1T45, IC4 74LVC1T45, IC5 74LVC1T45, IC6 ATXMEGA32A4U-AU, IC7 TPS73033DBV, Q1 BC807W-1907646, Q10 PMF280UN,115-1758094, Q11 PDTC123YU-1757992, Q2 NX2301P-1894738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

Commit message: shupito23: updated Farnell OC for 2.2uF
Parts:
- C3: value 2.2u-1759473 -> 2.2u
Changed lines of the file:
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@@
 <grid distance="0.3175" unitdist="mm" unit="mm" style="lines" multiple="1" display="yes" altdistance="0.003125" altunitdist="inch" altunit="inch"/>
 <layers>
-<layer number="1" name="Top" color="4" fill="1" visible="no" active="yes"/>
-<layer number="16" name="Bottom" color="1" fill="1" visible="no" active="yes"/>
-<layer number="17" name="Pads" color="2" fill="1" visible="no" active="yes"/>
-<layer number="18" name="Vias" color="2" fill="1" visible="no" active="yes"/>
+<layer number="1" name="Top" color="4" fill="1" visible="yes" active="yes"/>
+<layer number="16" name="Bottom" color="1" fill="1" visible="yes" active="yes"/>
+<layer number="17" name="Pads" color="2" fill="1" visible="yes" active="yes"/>
+<layer number="18" name="Vias" color="2" fill="1" visible="yes" active="yes"/>
 <layer number="19" name="Unrouted" color="6" fill="1" visible="no" active="yes"/>
-<layer number="20" name="Dimension" color="15" fill="1" visible="no" active="yes"/>
+<layer number="20" name="Dimension" color="15" fill="1" visible="yes" active="yes"/>
 <layer number="21" name="tPlace" color="7" fill="1" visible="no" active="yes"/>
 <layer number="22" name="bPlace" color="7" fill="1" visible="no" active="yes"/>
@@
 <layer number="98" name="Guide" color="6" fill="1" visible="no" active="no"/>
 <layer number="100" name="Drawings" color="4" fill="0" visible="no" active="yes"/>
-<layer number="101" name="FrontPrint" color="15" fill="1" visible="yes" active="yes"/>
+<layer number="101" name="FrontPrint" color="15" fill="1" visible="no" active="yes"/>
 <layer number="200" name="200bmp" color="7" fill="1" visible="no" active="yes"/>
 <layer number="250" name="Descript" color="7" fill="1" visible="no" active="yes"/>
@@
 <element name="JP9" library="pinhead_smd" package="PINH1X01SMD" value="PINH1X01SMD" x="41.91" y="1.905" rot="R270"/>
 <element name="JP10" library="pinhead_smd" package="PINH1X01SMD" value="PINH1X01SMD" x="41.91" y="1.905" rot="MR90"/>
-<element name="C3" library="rcl" package="C0603K" value="2.2u-1759473" x="19.05" y="4.445" rot="MR0"/>
+<element name="C3" library="rcl" package="C0603K" value="2.2u" x="19.05" y="4.445" rot="MR0"/>
 <element name="S1" library="switch" package="KSS-G" value="KSS241G" x="39.608125" y="19.05" rot="MR90"/>
 <element name="R3" library="rcl" package="R1206" value="0" x="34.29" y="3.175" rot="MR315"/>
