File: shupito23/shupito.sch (EAGLE design)
At the start: 92 parts, among them IC2 74LVC1T45, IC3 74LVC1T45, IC4 74LVC1T45, IC5 74LVC1T45, IC6 ATXMEGA32A4U-AU, IC7 TPS73033DBV, Q1 BC807W-1907646, Q10 PMF280UN,115-1758094, Q11 PDTC123YU-1757992, Q2 NX2301P-1894738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

Commit message: shupito23: Selected better transistors for the rst pin.
Parts:
- Q6, Q9: value DTA144-1680214 -> PDTA114TU-8736731
Changed lines of the file:
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@@
 <part name="R1" library="rcl" deviceset="R-EU_" device="R0603" value="330"/>
 <part name="R2" library="rcl" deviceset="R-EU_" device="R0603" value="6k8"/>
-<part name="Q9" library="transistors" deviceset="PNP-BIAS" device="-SOT323-BEC" value="DTA144-1680214"/>
+<part name="Q9" library="transistors" deviceset="PNP-BIAS" device="-SOT323-BEC" value="PDTA114TU-8736731"/>
 <part name="R13" library="rcl" deviceset="R-EU_" device="R0603" value="22k 1%"/>
 <part name="R14" library="rcl" deviceset="R-EU_" device="R0603" value="1k5 1%"/>
@@
 <part name="P+1" library="supply1" deviceset="+5V" device=""/>
 <part name="P+3" library="supply1" deviceset="+5V" device=""/>
-<part name="Q6" library="transistors" deviceset="PNP-BIAS" device="-SOT323-BEC" value="DTA144-1680214"/>
+<part name="Q6" library="transistors" deviceset="PNP-BIAS" device="-SOT323-BEC" value="PDTA114TU-8736731"/>
 <part name="Q11" library="transistors" deviceset="NPN-BIAS" device="-SOT323-BEC" value="PDTC123YU-1757992"/>
 <part name="VCC6" library="supply1" deviceset="VCCIO" device=""/>

Commit message: shupito23: updated Farnell OC for 2.2uF
Parts:
- C3: value 2.2u-1759473 -> 2.2u
Changed lines of the file:
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@@
 <part name="JP9" library="pinhead_smd" deviceset="PINH1X01" device="SMD"/>
 <part name="JP10" library="pinhead_smd" deviceset="PINH1X01" device="SMD"/>
-<part name="C3" library="rcl" deviceset="C-EU" device="C0603K" value="2.2u-1759473"/>
+<part name="C3" library="rcl" deviceset="C-EU" device="C0603K" value="2.2u"/>
 <part name="S1" library="switch" deviceset="KSS" device="G" technology="241"/>
 <part name="GND8" library="supply1" deviceset="GND" device=""/>
